File: hardware/backplane/5V_Buck.kicad_sch (KiCad schematic)
At the start: 18 parts, among them U2 TPS5450DDAR

Commit message: Update backplane design and previews
Parts:
- R11: footprint Resistor_SMD:R_0603_1608Metric -> Resistor_SMD:R_1206_3216Metric
Changed lines of the file:
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@@
 			)
 		)
-		(property "Footprint" "Resistor_SMD:R_0603_1608Metric"
+		(property "Footprint" "Resistor_SMD:R_1206_3216Metric"
 			(at 242.316 92.456 90)
 			(hide yes)
