File: hardware/backplane/HackerfabBackplane.kicad_pcb (KiCad board)
At the start: 2 copper layers, 93 parts, among them J1 9001-12961C00A, J2 9001-12961C00A, J3 9001-12961C00A, U1 TPS5450DDAR, U2 TPS5450DDAR, U3 AP2112K-3.3TRG1, U4 USBLC6-2SC6, U5 RP2354B, U6 TPS2116DRL, Y1 12MHz

Commit message: Update backplane design and previews
Parts:
- added D10: KT-0603R, Hack_Opto:LED_0603_1608Metric, F.Cu at (117.0, 151.2)
- added D7: TVS2700DRVR, Hack_Diodes:WSON-6_TVS2700DRV_2x2mm, F.Cu at (78.5, 126.5)
- added D8: BZT52C12 12V, Hack_Diodes:D_SOD-123, F.Cu at (73.0, 132.5)
- added D9: KT-0603R, Hack_Opto:LED_0603_1608Metric, F.Cu at (114.0, 151.2)
- added F1: 5A 125V, Hack_Passives:Fuse_Littelfuse-NANO2-451_453, F.Cu at (62.5, 124.0)
- added J4: KF128-5.08-2P-AA, Hack_Connector:KF128-5.08-2P-AA, F.Cu at (52.0, 128.0)
- added J5: KF128-5.08-2P-AA, Hack_Connector:KF128-5.08-2P-AA, F.Cu at (52.0, 145.0)
- added J6: KF128-5.08-2P-AA, Hack_Connector:KF128-5.08-2P-AA, F.Cu at (68.5, 178.1)
- added J7: TYPE-C-31-M-12, Hack_Connector:USB_C_Receptacle_HRO_TYPE-C-31-M-12, F.Cu at (135.0, 180.9)
- added J9: ZX-SH1.0-3PWT, Hack_Connector:Megastar_ZX-SH1.0-3PWT_1x03_P1.00mm_Horizontal, F.Cu at (154.5, 152.5)
- added Q1: DMP6023LE-13, Hack_Chips:SOT-223-3_TabPin4, F.Cu at (70.0, 126.5)
- added R20: 1k13, Resistor_SMD:R_0603_1608Metric, F.Cu at (69.5, 132.5)
- added R21: 1k13, Resistor_SMD:R_0603_1608Metric, F.Cu at (69.5, 135.5)
- added R22: 5k1, Resistor_SMD:R_0603_1608Metric, F.Cu at (138.3, 173.0)
- added R23: 5k1, Resistor_SMD:R_0603_1608Metric, F.Cu at (131.0, 175.0)
- added R24: 100R, Resistor_SMD:R_0603_1608Metric, F.Cu at (146.7, 153.5)
- added R25: 100R, Resistor_SMD:R_0603_1608Metric, F.Cu at (146.7, 151.5)
- added R26: 0R, Resistor_SMD:R_0402_1005Metric, F.Cu at (139.0, 170.5)
- added R27: 0R, Resistor_SMD:R_0402_1005Metric, F.Cu at (140.5, 170.5)
- added R28: 0R, Resistor_SMD:R_0402_1005Metric, F.Cu at (143.5, 171.5)
- added R29: 0R, Resistor_SMD:R_0402_1005Metric, F.Cu at (143.5, 170.5)
- added R30: 0R, Resistor_SMD:R_0402_1005Metric, F.Cu at (143.5, 169.5)
- added R31: 0R, Resistor_SMD:R_0402_1005Metric, F.Cu at (143.5, 168.5)
- added R32: 0R, Resistor_SMD:R_0402_1005Metric, F.Cu at (145.5, 141.5)
- added R33: 0R, Resistor_SMD:R_0402_1005Metric, F.Cu at (138.0, 141.5)
- added R34: 0R, Resistor_SMD:R_0402_1005Metric, F.Cu at (143.5, 141.5)
- added R35: 0R, Resistor_SMD:R_0402_1005Metric, F.Cu at (144.5, 141.5)
- added R36: 0R, Resistor_SMD:R_0402_1005Metric, F.Cu at (137.0, 141.5)
- added R37: 0R, Resistor_SMD:R_0402_1005Metric, F.Cu at (136.0, 141.5)
- added R38: 0R, Resistor_SMD:R_0402_1005Metric, F.Cu at (143.5, 167.5)
- added R39: 0R, Resistor_SMD:R_0402_1005Metric, F.Cu at (147.5, 160.5)
- added R40: 0R, Resistor_SMD:R_0402_1005Metric, F.Cu at (143.5, 165.5)
- added R41: 0R, Resistor_SMD:R_0402_1005Metric, F.Cu at (143.5, 166.5)
- added R42: 0R, Resistor_SMD:R_0402_1005Metric, F.Cu at (143.5, 164.5)
- added R43: 0R, Resistor_SMD:R_0402_1005Metric, F.Cu at (143.5, 163.5)
- added R44: 0R, Resistor_SMD:R_0402_1005Metric, F.Cu at (118.0, 160.5)
- added R45: 0R, Resistor_SMD:R_0402_1005Metric, F.Cu at (118.0, 162.0)
- added R46: 0R, Resistor_SMD:R_0402_1005Metric, F.Cu at (118.0, 163.5)
- added R47: 0R, Resistor_SMD:R_0402_1005Metric, F.Cu at (135.0, 141.5)
- added R48: 0R, Resistor_SMD:R_0402_1005Metric, F.Cu at (134.0, 141.5)
- added R49: 0R, Resistor_SMD:R_0402_1005Metric, F.Cu at (133.0, 141.5)
- added R50: 0R, Resistor_SMD:R_0402_1005Metric, F.Cu at (132.0, 141.5)
- added R51: 0R, Resistor_SMD:R_0402_1005Metric, F.Cu at (131.0, 141.5)
- added R52: 0R, Resistor_SMD:R_0402_1005Metric, F.Cu at (130.0, 141.5)
- added R53: 1k13, Resistor_SMD:R_0603_1608Metric, F.Cu at (114.0, 147.3)
- added R54: 1k13, Resistor_SMD:R_0603_1608Metric, F.Cu at (117.0, 147.5)
- added TP10: ~, TestPoint:TestPoint_Pad_1.0x1.0mm, F.Cu at (52.0, 120.0)
- added TP11: ~, TestPoint:TestPoint_Pad_1.0x1.0mm, F.Cu at (75.5, 127.0)
- added TP12: ~, TestPoint:TestPoint_Pad_1.0x1.0mm, F.Cu at (67.5, 132.0)
- R11, R6: footprint Resistor_SMD:R_0603_1608Metric -> Resistor_SMD:R_1206_3216Metric
- moved H4 94.8 mm to (154.0, 180.5), turned to 180 degrees
- moved H3 89.7 mm to (49.5, 180.5), turned to 90 degrees
- moved U6 87.8 mm to (103.2, 173.8)
- moved U3 84.9 mm to (115.5, 171.6), turned to -90 degrees
- moved C40 84.0 mm to (99.0, 172.5), turned to 90 degrees
- moved C39 83.9 mm to (100.5, 172.5), turned to 90 degrees
- moved D6 83.8 mm to (118.2, 178.2), turned to -90 degrees
- moved C37 83.6 mm to (107.0, 176.5), turned to -90 degrees
- moved TP9 82.8 mm to (105.0, 171.0)
- moved R12 82.4 mm to (115.7, 178.3), turned to -90 degrees
- moved C16 81.8 mm to (115.8, 174.8), turned to 180 degrees
- moved R19 81.1 mm to (101.5, 176.0), turned to 180 degrees
- moved C15 80.7 mm to (114.8, 168.8)
- moved R18 79.7 mm to (104.5, 176.0), turned to 180 degrees
- moved C38 79.5 mm to (107.0, 172.0), turned to 90 degrees
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Connections:
- net +24V renamed +24V_P
- net /USB Voltage MUX/5V_USB renamed +5V_USB
- U4 pad 1: /Microcontroller/USB_D- -> /USB_D-
- U4 pad 3: /Microcontroller/USB_D+ -> /USB_D+
- U5 pad 1: unconnected-(U5-GPIO4-Pad1) -> Net-(U5-GPIO4)
- U5 pad 11: unconnected-(U5-GPIO12-Pad11) -> Net-(U5-GPIO12)
- U5 pad 12: unconnected-(U5-GPIO13-Pad12) -> Net-(U5-GPIO13)
- U5 pad 16: unconnected-(U5-GPIO16-Pad16) -> Net-(U5-GPIO16)
- U5 pad 17: unconnected-(U5-GPIO17-Pad17) -> Net-(U5-GPIO17)
- U5 pad 18: unconnected-(U5-GPIO18-Pad18) -> Net-(U5-GPIO18)
- U5 pad 19: unconnected-(U5-GPIO19-Pad19) -> Net-(U5-GPIO19)
- U5 pad 2: unconnected-(U5-GPIO5-Pad2) -> Net-(U5-GPIO5)
- U5 pad 20: unconnected-(U5-GPIO20-Pad20) -> Net-(U5-GPIO20)
- U5 pad 21: unconnected-(U5-GPIO21-Pad21) -> Net-(U5-GPIO21)
- U5 pad 22: unconnected-(U5-GPIO22-Pad22) -> Net-(U5-GPIO22)
- U5 pad 23: unconnected-(U5-GPIO23-Pad23) -> Net-(U5-GPIO23)
- U5 pad 25: unconnected-(U5-GPIO24-Pad25) -> Net-(U5-GPIO24)
- U5 pad 26: unconnected-(U5-GPIO25-Pad26) -> Net-(U5-GPIO25)
- U5 pad 27: unconnected-(U5-GPIO26-Pad27) -> Net-(U5-GPIO26)
- U5 pad 28: unconnected-(U5-GPIO27-Pad28) -> Net-(U5-GPIO27)
- U5 pad 3: unconnected-(U5-GPIO6-Pad3) -> Net-(U5-GPIO6)
- U5 pad 33: /Microcontroller/SWCLK -> Net-(U5-SWCLK)
- U5 pad 34: /Microcontroller/SWDIO -> Net-(U5-SWDIO)
- U5 pad 36: unconnected-(U5-GPIO28-Pad36) -> Net-(U5-GPIO28)
- U5 pad 37: unconnected-(U5-GPIO29-Pad37) -> Net-(U5-GPIO29)
- U5 pad 4: unconnected-(U5-GPIO7-Pad4) -> Net-(U5-GPIO7)
- U5 pad 49: unconnected-(U5-GPIO40/ADC0-Pad49) -> Net-(U5-GPIO40/ADC0)
- U5 pad 52: unconnected-(U5-GPIO41/ADC1-Pad52) -> Net-(U5-GPIO41/ADC1)
- U5 pad 53: unconnected-(U5-GPIO42/ADC2-Pad53) -> Net-(U5-GPIO42/ADC2)
- U5 pad 6: unconnected-(U5-GPIO8-Pad6) -> Net-(U5-GPIO8)
- U5 pad 7: unconnected-(U5-GPIO9-Pad7) -> Net-(U5-GPIO9)
- U5 pad 77: unconnected-(U5-GPIO0-Pad77) -> Net-(U5-GPIO0)
- U5 pad 78: unconnected-(U5-GPIO1-Pad78) -> Net-(U5-GPIO1)
- U5 pad 8: unconnected-(U5-GPIO10-Pad8) -> Net-(U5-GPIO10)
- U5 pad 9: unconnected-(U5-GPIO11-Pad9) -> Net-(U5-GPIO11)
Other:
- board outline added: 111.5 x 142 mm

Commit message: Update backplane and libraries from October 29 archives
Import the supplied active KiCad sources, retain portable library tables, and omit local editor state. Refresh schematic and board previews, archive fingerprints, and validation notes for the partially routed 144-component design.
Parts:
- added C41: 100n 50V, Capacitor_SMD:C_0402_1005Metric, F.Cu at (141.7, 182.3)
- added U7: W25Q128JVSIQ, Hack_Chips:W25Q128JVSIQ_SOIC-8_5.3x5.3mm_P1.27mm, F.Cu at (139.1, 177.0)
- L3: value 3.3u -> 3.3uH; footprint Hack_Passives:coilcraft_lps4018_dot1 -> Hack_Passives:L_Murata_DFE252012F_2.5x2.0mm
- moved C17 30.9 mm to (120.8, 167.8), turned to 180 degrees
- moved D6 22.6 mm to (102.7, 161.8), turned to 0 degrees
- moved R23 22.4 mm to (109.0, 179.2), turned to -90 degrees
- moved C15 21.8 mm to (93.3, 165.2), turned to 90 degrees
- moved U3 20.6 mm to (96.2, 164.5), turned to 0 degrees
- moved C16 19.6 mm to (99.3, 164.2), turned to -90 degrees
- moved J7 19.4 mm to (115.6, 180.3)
- moved R12 19.1 mm to (102.8, 164.3), turned to 0 degrees
- moved R22 17.2 mm to (122.2, 179.0), turned to -90 degrees
- moved R53 12.4 mm to (118.6, 158.8), turned to 180 degrees
- moved H1 12.0 mm to (49.5, 33.6)
- moved H2 12.0 mm to (154.0, 33.6)
- moved J1 11.6 mm to (62.4, 53.0)
- moved R54 9.05 mm to (118.7, 156.4), turned to 180 degrees
- moved J2 8.58 mm to (62.5, 79.0)
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Connections:
- net Net-(U5-~{QSPI_SS}) renamed /Microcontroller/~{QSPI_SS}
- J1 pad B25: GND -> +5V
- J1 pad B26: GND -> +5V
- J1 pad B28: GND -> +12V
- J1 pad B29: GND -> +12V
- J1 pad B4: GND -> +12V
- J1 pad B5: GND -> +12V
- J1 pad B7: GND -> +5V
- J1 pad B8: GND -> +5V
- J2 pad B25: GND -> +5V
- J2 pad B26: GND -> +5V
- J2 pad B28: GND -> +12V
- J2 pad B29: GND -> +12V
- J2 pad B4: GND -> +12V
- J2 pad B5: GND -> +12V
- J2 pad B7: GND -> +5V
- J2 pad B8: GND -> +5V
- J3 pad B25: GND -> +5V
- J3 pad B26: GND -> +5V
- J3 pad B28: GND -> +12V
- J3 pad B29: GND -> +12V
- J3 pad B4: GND -> +12V
- J3 pad B5: GND -> +12V
- J3 pad B7: GND -> +5V
- J3 pad B8: GND -> +5V
- R26 pad 1: /Microcontroller/UART_TX -> /UART_TX
- R27 pad 1: /Microcontroller/UART_RX -> /UART_RX
- R28 pad 1: /Microcontroller/I2C0_SDA -> /I2C0_SDA
- R29 pad 1: /Microcontroller/I2C0_SCL -> /I2C0_SCL
- R30 pad 1: /Microcontroller/I2C1_SDA -> /I2C1_SDA
- R31 pad 1: /Microcontroller/I2C1_SCL -> /I2C1_SCL
- R32 pad 1: /Microcontroller/SPI0_MISO -> /SPI0_MISO
- R33 pad 1: /Microcontroller/SPI0_MOSI -> /SPI0_MOSI
- R34 pad 1: /Microcontroller/SPI0_CLK -> /SPI0_CLK
- R35 pad 1: /Microcontroller/SPI0_CS1 -> /SPI0_CS1
- R36 pad 1: /Microcontroller/SPI0_CS2 -> /SPI0_CS2
- R37 pad 1: /Microcontroller/SPI0_CS3 -> /SPI0_CS3
- R38 pad 1: /Microcontroller/SPI1_MISO -> /SPI1_MISO
- R39 pad 1: /Microcontroller/SPI1_MOSI -> /SPI1_MOSI
- R40 pad 1: /Microcontroller/SPI1_CLK -> /SPI1_CLK
- R41 pad 1: /Microcontroller/SPI1_CS1 -> /SPI1_CS1
- R42 pad 1: /Microcontroller/SPI1_CS2 -> /SPI1_CS2
- R43 pad 1: /Microcontroller/SPI1_CS3 -> /SPI1_CS3
- R44 pad 1: /Microcontroller/AUX1 -> /AUX1
- R45 pad 1: /Microcontroller/AUX4 -> /AUX4
- R46 pad 1: /Microcontroller/AUX7 -> /AUX7
- R47 pad 1: /Microcontroller/AUX2 -> /AUX2
- R48 pad 1: /Microcontroller/AUX3 -> /AUX3
- R49 pad 1: /Microcontroller/AUX5 -> /AUX5
- R50 pad 1: /Microcontroller/AUX6 -> /AUX6
- R51 pad 1: /Microcontroller/AUX8 -> /AUX8
- R52 pad 1: /Microcontroller/AUX9 -> /AUX9
- R53 pad 1: Net-(U5-GPIO29) -> Net-(U5-GPIO34)
- R54 pad 1: Net-(U5-GPIO28) -> Net-(U5-GPIO33)
- U5 pad 36: Net-(U5-GPIO28) -> unconnected-(U5-GPIO28-Pad36)
- U5 pad 37: Net-(U5-GPIO29) -> unconnected-(U5-GPIO29-Pad37)
- U5 pad 42: unconnected-(U5-GPIO33-Pad42) -> Net-(U5-GPIO33)
- U5 pad 43: unconnected-(U5-GPIO34-Pad43) -> Net-(U5-GPIO34)
- U5 pad 70: unconnected-(U5-QSPI_SD3-Pad70) -> /Microcontroller/QSPI_SD3
- U5 pad 71: unconnected-(U5-QSPI_SCLK-Pad71) -> /Microcontroller/QSPI_SCLK
- U5 pad 72: unconnected-(U5-QSPI_SD0-Pad72) -> /Microcontroller/QSPI_SD0
- U5 pad 73: unconnected-(U5-QSPI_SD2-Pad73) -> /Microcontroller/QSPI_SD2
- U5 pad 74: unconnected-(U5-QSPI_SD1-Pad74) -> /Microcontroller/QSPI_SD1
Routing:
- net GND: track 0.00 -> 67.0 mm, vias 0 -> 85
- net /Microcontroller/~{QSPI_SS}: track 0.00 -> 57.7 mm
- net +3V3: track 0.00 -> 44.0 mm, vias 0 -> 4
- net Net-(U5-RUN): track 0.00 -> 33.6 mm
- net Net-(U5-SWDIO): track 0.00 -> 25.0 mm, vias 0 -> 2
- net +24V_P: track 0.00 -> 24.6 mm, vias 0 -> 13
- net Net-(U5-SWCLK): track 0.00 -> 23.7 mm, vias 0 -> 2
- net Net-(U5-GPIO23): track 0.00 -> 23.7 mm, vias 0 -> 2
- net /Microcontroller/QSPI_SD3: track 0.00 -> 23.3 mm
- net Net-(U5-GPIO26): track 0.00 -> 22.9 mm, vias 0 -> 2
- net Net-(U5-GPIO24): track 0.00 -> 22.8 mm, vias 0 -> 2
- net Net-(U5-GPIO27): track 0.00 -> 21.8 mm, vias 0 -> 2
- net Net-(U5-GPIO16): track 0.00 -> 21.7 mm
- net Net-(U5-GPIO17): track 0.00 -> 21.1 mm
- net Net-(U5-GPIO25): track 0.00 -> 20.8 mm
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- added copper zone on F.Cu, net +12V
- added copper zone on In2.Cu, net +12V
- added copper zone on In2.Cu, net +1V1
- added copper zone on F.Cu, net +24V
- added copper zone on F.Cu, net +24V_P
- added copper zone on In2.Cu, net +24V_P
- added copper zone on In2.Cu, net +3V3
- added copper zone on F.Cu, net +5V
- added copper zone on In2.Cu, net +5V
- added copper zone on F.Cu, net /5V Buck Regulator/5V_BUCK
- added copper zone on In2.Cu, net /5V Buck Regulator/5V_BUCK
- added copper zone on F.Cu, net GND
- added copper zone on In1.Cu, net GND
- added copper zone on F.Cu, net Net-(C12-Pad1)
- added copper zone on F.Cu, net Net-(C5-Pad1)
- added copper zone on F.Cu, net Net-(D2-K)
- added copper zone on F.Cu, net Net-(D4-K)
- added copper zone on F.Cu, net Net-(F1-Pad1)
Other:
- board size 111.5 x 142 mm -> 111.5 x 154 mm
- copper layers 2 -> 4
- board text added: "SN:"
