File: hardware/backplane/HackerfabBackplane.kicad_pcb (KiCad board)
At the start: 4 copper layers, 111.5 x 154 mm, 144 parts, among them J1 9001-12961C00A, J2 9001-12961C00A, J3 9001-12961C00A, J4 KF128-5.08-2P-AA, J5 KF128-5.08-2P-AA, J6 KF128-5.08-2P-AA, J7 TYPE-C-31-M-12, J9 ZX-SH1.0-3PWT, Q1 DMP6023LE-13, U1 TPS5450DDAR, U2 TPS5450DDAR, U3 AP2112K-3.3TRG1, U4 USBLC6-2SC6, U5 RP2354B, U6 TPS2116DRL, U7 W25Q128JVSIQ, Y1 12MHz

Commit message: Arrange connector signals around the MCU jumper banks
Keep each protocol paired across A/C columns and UART RX/TX together. Update schematic and PCB signal assignments, add pin tables and a top-layer passage guide, and verify fixed power/ground, signal inventory, source jumpers, and KiCad parity.
Connections:
- J1 pad A10: /I2C1_SDA -> unconnected-(J1-PadA10)
- J1 pad A11: /SPI0_MISO -> /AUX1
- J1 pad A12: /SPI0_MOSI -> unconnected-(J1-PadA12)
- J1 pad A13: /SPI0_CLK -> unconnected-(J1-PadA13)
- J1 pad A14: /SPI1_MISO -> /AUX2
- J1 pad A15: /SPI1_MOSI -> /SPI0_CS3
- J1 pad A16: /SPI1_CLK -> /SPI0_MOSI
- J1 pad A17: unconnected-(J1-PadA17) -> /SPI0_CS1
- J1 pad A18: unconnected-(J1-PadA18) -> /SPI1_CS3
- J1 pad A19: unconnected-(J1-PadA19) -> /SPI1_MOSI
- J1 pad A20: /AUX3 -> /SPI1_CS1
- J1 pad A21: /AUX1 -> /I2C1_SCL
- J1 pad A22: /UART_TX -> /I2C0_SCL
- J1 pad A23: /I2C0_SDA -> /UART_RX
- J1 pad C10: /I2C1_SCL -> unconnected-(J1-PadC10)
- J1 pad C11: /SPI0_CS1 -> unconnected-(J1-PadC11)
- J1 pad C12: /SPI0_CS2 -> unconnected-(J1-PadC12)
- J1 pad C13: /SPI0_CS3 -> /AUX3
- J1 pad C14: /SPI1_CS1 -> unconnected-(J1-PadC14)
- J1 pad C15: /SPI1_CS2 -> /SPI0_CS2
- J1 pad C16: /SPI1_CS3 -> /SPI0_CLK
- J1 pad C17: unconnected-(J1-PadC17) -> /SPI0_MISO
- J1 pad C18: unconnected-(J1-PadC18) -> /SPI1_CS2
- J1 pad C19: unconnected-(J1-PadC19) -> /SPI1_CLK
- J1 pad C20: unconnected-(J1-PadC20) -> /SPI1_MISO
- J1 pad C21: /AUX2 -> /I2C1_SDA
- J1 pad C22: /UART_RX -> /I2C0_SDA
- J1 pad C23: /I2C0_SCL -> /UART_TX
- J2 pad A10: /I2C1_SDA -> unconnected-(J2-PadA10)
- J2 pad A11: /SPI0_MISO -> unconnected-(J2-PadA11)
- J2 pad A12: /SPI0_MOSI -> unconnected-(J2-PadA12)
- J2 pad A13: /SPI0_CLK -> /AUX5
- J2 pad A14: /SPI1_MISO -> unconnected-(J2-PadA14)
- J2 pad A15: /SPI1_MOSI -> /SPI0_CS3
- J2 pad A16: /SPI1_CLK -> /SPI0_MOSI
- J2 pad A17: unconnected-(J2-PadA17) -> /SPI0_CS1
- J2 pad A18: unconnected-(J2-PadA18) -> /SPI1_CS3
- J2 pad A19: /AUX5 -> /SPI1_MOSI
- J2 pad A20: unconnected-(J2-PadA20) -> /SPI1_CS1
- J2 pad A21: unconnected-(J2-PadA21) -> /I2C1_SCL
- J2 pad A22: unconnected-(J2-PadA22) -> /I2C0_SCL
- J2 pad A23: /I2C0_SDA -> unconnected-(J2-PadA23)
- J2 pad C10: /I2C1_SCL -> /AUX4
- J2 pad C11: /SPI0_CS1 -> unconnected-(J2-PadC11)
- J2 pad C12: /SPI0_CS2 -> /AUX6
- J2 pad C13: /SPI0_CS3 -> unconnected-(J2-PadC13)
- J2 pad C14: /SPI1_CS1 -> unconnected-(J2-PadC14)
- J2 pad C15: /SPI1_CS2 -> /SPI0_CS2
- J2 pad C16: /SPI1_CS3 -> /SPI0_CLK
- J2 pad C17: unconnected-(J2-PadC17) -> /SPI0_MISO
- J2 pad C18: unconnected-(J2-PadC18) -> /SPI1_CS2
- J2 pad C19: /AUX6 -> /SPI1_CLK
- J2 pad C20: /AUX4 -> /SPI1_MISO
- J2 pad C21: unconnected-(J2-PadC21) -> /I2C1_SDA
- J2 pad C22: unconnected-(J2-PadC22) -> /I2C0_SDA
- J2 pad C23: /I2C0_SCL -> unconnected-(J2-PadC23)
- J3 pad A10: /I2C1_SDA -> /AUX7
- J3 pad A11: /SPI0_MISO -> unconnected-(J3-PadA11)
- J3 pad A12: /SPI0_MOSI -> /AUX8
- J3 pad A13: /SPI0_CLK -> unconnected-(J3-PadA13)
- J3 pad A14: /SPI1_MISO -> unconnected-(J3-PadA14)
- J3 pad A15: /SPI1_MOSI -> /SPI0_CS3
- J3 pad A16: /SPI1_CLK -> /SPI0_MOSI
- J3 pad A17: /AUX9 -> /SPI0_CS1
- J3 pad A18: /AUX7 -> /SPI1_CS3
- J3 pad A19: unconnected-(J3-PadA19) -> /SPI1_MOSI
- J3 pad A20: unconnected-(J3-PadA20) -> /SPI1_CS1
- J3 pad A21: unconnected-(J3-PadA21) -> /I2C1_SCL
- J3 pad A22: unconnected-(J3-PadA22) -> /I2C0_SCL
- J3 pad A23: /I2C0_SDA -> /UART_RX
- J3 pad C10: /I2C1_SCL -> unconnected-(J3-PadC10)
- J3 pad C11: /SPI0_CS1 -> /AUX9
- J3 pad C12: /SPI0_CS2 -> unconnected-(J3-PadC12)
- J3 pad C13: /SPI0_CS3 -> unconnected-(J3-PadC13)
- J3 pad C14: /SPI1_CS1 -> /AUX10
- J3 pad C15: /SPI1_CS2 -> /SPI0_CS2
- J3 pad C16: /SPI1_CS3 -> /SPI0_CLK
- J3 pad C17: /AUX10 -> /SPI0_MISO
- J3 pad C18: /AUX8 -> /SPI1_CS2
- J3 pad C19: unconnected-(J3-PadC19) -> /SPI1_CLK
- J3 pad C20: unconnected-(J3-PadC20) -> /SPI1_MISO
- J3 pad C21: unconnected-(J3-PadC21) -> /I2C1_SDA
- J3 pad C22: /UART_RX -> /I2C0_SDA
- J3 pad C23: /I2C0_SCL -> unconnected-(J3-PadC23)
