File: hardware/backplane/Microcontroller.kicad_sch (KiCad schematic)
At the start: 35 parts, among them U4 USBLC6-2SC6, U5 RP2354B, Y1 12MHz

Commit message: Update backplane design and previews
Parts:
- added D10, D9: KT-0603R, Hack_Opto:LED_0603_1608Metric, symbol Hack_Opto:KT-0603R
- added R24, R25: 100R, Resistor_SMD:R_0603_1608Metric, symbol Hack_Passives:RNCP0603FTD100R
- added R26, R27, R28, R29, R30, R31, R32, R33, R34, R35, R36, R37, R38, R39, R40, R41, R42, R43, R44, R45, R46, R47, R48, R49, R50, R51, R52: 0R, Resistor_SMD:R_0402_1005Metric, symbol Hack_Passives:AA0402JR-070RL
- added R53, R54: 1k13, Resistor_SMD:R_0603_1608Metric, symbol Hack_Passives:RT0603FRE071K13L
Connections:
- net GND: now also D10.1 (K), D9.1 (K)
- net SWCLK: now also R24.2; no longer U5.33 (SWCLK)
- net SWDIO: now also R25.2; no longer U5.34 (SWDIO)
- net at U5.1 (GPIO4): now also R28.2
- net at U5.11 (GPIO12): now also R42.2
- net at U5.12 (GPIO13): now also R43.2
- net at U5.16 (GPIO16): now also R32.2
- net at U5.17 (GPIO17): now also R35.2
- net at U5.18 (GPIO18): now also R34.2
- net at U5.19 (GPIO19): now also R33.2
- net at U5.2 (GPIO5): now also R29.2
- net at U5.20 (GPIO20): now also R36.2
- net at U5.21 (GPIO21): now also R37.2
- net at U5.22 (GPIO22): now also R47.2
- net at U5.23 (GPIO23): now also R48.2
- net at U5.25 (GPIO24): now also R49.2
- net at U5.26 (GPIO25): now also R50.2
- net at U5.27 (GPIO26): now also R51.2
- net at U5.28 (GPIO27): now also R52.2
- net at U5.3 (GPIO6): now also R30.2
- net at U5.36 (GPIO28): now also R54.1
- net at U5.37 (GPIO29): now also R53.1
- net at U5.4 (GPIO7): now also R31.2
- net at U5.49 (GPIO40/ADC0): now also R44.2
- net at U5.52 (GPIO41/ADC1): now also R45.2
- net at U5.53 (GPIO42/ADC2): now also R46.2
- net at U5.6 (GPIO8): now also R38.2
- net at U5.7 (GPIO9): now also R41.2
- net at U5.77 (GPIO0): now also R26.2
- net at U5.78 (GPIO1): now also R27.2
- net at U5.8 (GPIO10): now also R40.2
- net at U5.9 (GPIO11): now also R39.2
- new net: D10.2 (A), R54.2
- new net: D9.2 (A), R53.2
- new net: R25.1, U5.34 (SWDIO)
- new net: R24.1, U5.33 (SWCLK)
- new net AUX1: R44.1
- new net AUX2: R47.1
- new net AUX3: R48.1
- new net AUX4: R45.1
- new net AUX5: R49.1
- new net AUX6: R50.1
- new net AUX7: R46.1
- new net AUX8: R51.1
- new net AUX9: R52.1
- new net I2C0_SCL: R29.1
- new net I2C0_SDA: R28.1
- new net I2C1_SCL: R31.1
- new net I2C1_SDA: R30.1
- new net SPI0_CLK: R34.1
- new net SPI0_CS1: R35.1
- new net SPI0_CS2: R36.1
- new net SPI0_CS3: R37.1
- new net SPI0_MISO: R32.1
- new net SPI0_MOSI: R33.1
- new net SPI1_CLK: R40.1
- new net SPI1_CS1: R41.1
- new net SPI1_CS2: R42.1
- new net SPI1_CS3: R43.1
- new net SPI1_MISO: R38.1
- new net SPI1_MOSI: R39.1
- new net UART_RX: R27.1
- new net UART_TX: R26.1
- no-connect marks 5 -> 24

Commit message: Update backplane and libraries from October 29 archives
Import the supplied active KiCad sources, retain portable library tables, and omit local editor state. Refresh schematic and board previews, archive fingerprints, and validation notes for the partially routed 144-component design.
Parts:
- removed L3: 3.3u, Hack_Passives:coilcraft_lps4018_dot1, symbol Hack_Passives:LPS4018-332MRC_Evaluation
- added C41: 100n 50V, Capacitor_SMD:C_0402_1005Metric, symbol Hack_Passives:0402B104K500HI
- added L3: 3.3uH, Hack_Passives:L_Murata_DFE252012F_2.5x2.0mm, symbol Hack_Passives:DFE252012F-3R3M=P2
- added U7: W25Q128JVSIQ, Hack_Chips:W25Q128JVSIQ_SOIC-8_5.3x5.3mm_P1.27mm, symbol Hack_Chips:W25Q128JVSIQ
Connections:
- net +1V1: now also L3.1
- net +3V3: now also C41.1, U7.8 (VCC)
- net GND: now also C41.2, U7.4 (GND)
- net at U5.63 (VREG_LX): now also L3.2
- net at R54.1: now also U5.42 (GPIO33); no longer U5.36 (GPIO28)
- net ~{QSPI_SS}: now reaches R13.1, TP6.1, U5.75 (~{QSPI_SS})
- net ~{QSPI_SS}: now also U7.1 (~{CS})
- net at U5.37 (GPIO29): no longer R53.1
- net at U5.43 (GPIO34): now also R53.1
- net QSPI_SD3: now reaches U5.70 (QSPI_SD3)
- net QSPI_SD3: now also U7.7 (IO3)
- net QSPI_SCLK: now reaches U5.71 (QSPI_SCLK)
- net QSPI_SCLK: now also U7.6 (CLK)
- net QSPI_SD0: now reaches U5.72 (QSPI_SD0)
- net QSPI_SD0: now also U7.5 (IO0/DI)
- net QSPI_SD2: now reaches U5.73 (QSPI_SD2)
- net QSPI_SD2: now also U7.3 (IO2/~{WP})
- net QSPI_SD1: now reaches U5.74 (QSPI_SD1)
- net QSPI_SD1: now also U7.2 (IO1/DO)
- no-connect marks 24 -> 19
Other:
- moved on the sheet: D10, D9, R53, R54
